Commit message: save rviz config

File: src/rover/description/robot_core.xacro (robot description, xacro)
@@ -1,5 +1,5 @@
 <?xml version="1.0"?>
 <robot xmlns:xacro="http://www.ros.org/wiki/xacro">
-    <!-- <xacro:include filename="internal_macros.xacro" /> -->
+    <xacro:include filename="inertial_macros.xacro" />
     <material name="white">
     <color rgba="1 1 1 1"/>
@@ -38,4 +38,7 @@
             </geometry>
         </collision>
+        <xacro:inertial_box mass="0.3" x="0.3" y="0.3" z="0.15">
+            <origin xyz="0.15 0 0.075" rpy="0 0 0"/>
+        </xacro:inertial_box>
     </link>
 <!-- Left Wheel -->
@@ -55,7 +58,10 @@
         <collision>
             <geometry>
-                <cylinder length="0.05" radius="0.04" />
+                <cylinder length="0.04" radius="0.04" />
             </geometry>
         </collision>
+        <xacro:inertial_cylinder mass="0.1" length="0.05" radius="0.04">
+            <origin xyz="0 0 0" rpy="0 0 0"/>
+        </xacro:inertial_cylinder>
     </link>
 <!-- Right Wheel -->
@@ -79,4 +85,7 @@
             <material name="red"/>
         </collision>
+        <xacro:inertial_cylinder mass="0.1" length="0.05" radius="0.04">
+            <origin xyz="0 0 0" rpy="0 0 0"/>
+        </xacro:inertial_cylinder>
     </link>
 <!-- Caster wheel -->
@@ -98,4 +107,7 @@
             </geometry>
         </collision>
+        <xacro:inertial_sphere mass="0.1" radius="0.04">
+            <origin xyz="0 0 0" rpy="0 0 0"/>
+        </xacro:inertial_sphere>
     </link>
 </robot>
